File: right-pcb/right-pcb.kicad_pcb (KiCad board)
At the start: 2 copper layers, 255.3 x 104.6 mm, 82 parts, among them J1 BAT, J2 BAT, U1 xiao-ble, U2 xiao-ble

Commit message: Update right-pcb to rev 0.3
Parts:
- removed DL1, DL10, DL11, DL12, DL13, DL14, DL15, DL16, DL17, DL18, DL2, DL3, DL4, DL5, DL6, DL7, DL8, DL9: D_Small, karmalib:Diode_SOD123
- removed J1: BAT, karmalib:JST_PH_S2B-PH-SM4-TB
- removed the REF** at (131.8, 103.1)
- removed the REF** at (31.7, 113.5)
- removed the REF** at (131.8, 35.8)
- removed the REF** at (55.4, 35.8)
- removed RSW1: SW_Push, karmalib:SKHLLCA010
- removed SWL1, SWL10, SWL11, SWL12, SWL13, SWL14, SWL15, SWL16, SWL17, SWL18, SWL2, SWL3, SWL4, SWL5, SWL6, SWL7, SWL8, SWL9: SW_Push_45deg, karmalib:Kailh_Socket_PG1350_Optional
- removed U1: xiao-ble, karmalib:XIAO_nRF52840_SMD_Cutout
- added REF**: MountingHole_2.2mm_M2_DIN965_Pad, MountingHole:MountingHole_2.2mm_M2_DIN965_Pad, F.Cu at (59.9, 101.0)
- added REF**: MountingHole_2.2mm_M2_DIN965_Pad, MountingHole:MountingHole_2.2mm_M2_DIN965_Pad, F.Cu at (137.2, 35.9)
- added REF**: MountingHole_2.2mm_M2_DIN965_Pad, MountingHole:MountingHole_2.2mm_M2_DIN965_Pad, F.Cu at (158.9, 112.5)
- added REF**: MountingHole_2.2mm_M2_DIN965_Pad, MountingHole:MountingHole_2.2mm_M2_DIN965_Pad, F.Cu at (59.9, 35.9)
- moved RSW2 170.0 mm to (75.7, 37.3)
- moved SWR11 121.7 mm to (71.4, 90.1)
- moved SWR6 121.7 mm to (71.4, 71.1)
- moved SWR1 121.7 mm to (71.4, 52.1)
- moved DR11 121.6 mm to (63.4, 83.9)
- moved DR1 121.6 mm to (63.4, 45.9)
- moved DR6 121.6 mm to (63.4, 64.9)
- moved DR17 121.6 mm to (60.5, 109.1)
- moved U2 121.6 mm to (151.2, 43.1)
- moved DR16 121.3 mm to (40.6, 119.6)
- moved SWR12 121.2 mm to (90.4, 85.4)
- moved SWR7 121.2 mm to (90.4, 66.4)
- moved SWR2 121.2 mm to (90.4, 47.4)
- moved SWR18 121.2 mm to (90.4, 110.1)
- moved DR18 121.1 mm to (82.4, 103.9)
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Routing:
- net ROW3_R: track 0.15 -> 190.7 mm, vias 0 -> 4
- net COL4_R: track 0.21 -> 176.5 mm
- net ROW2_R: track 0.05 -> 165.8 mm, vias 0 -> 10
- net COL3_R: track 0.00 -> 147.9 mm
- net ROW1_R: track 0.05 -> 147.7 mm, vias 0 -> 10
- net COL2_R: track 1.13 -> 117.6 mm
- net ROW0_R: track 0.13 -> 103.4 mm, vias 0 -> 8
- net RESET_R: track 1.08 -> 87.0 mm
- net VBAT_R: track 0.00 -> 82.5 mm
- net COL0_R: track 0.70 -> 78.1 mm
- net COL1_R: track 0.00 -> 64.9 mm
- net Net-(DR1-A): track 0.26 -> 8.78 mm
- net Net-(DR16-A): track 0.00 -> 8.51 mm
- net Net-(DR17-A): track 0.00 -> 8.18 mm
- net Net-(DR5-A): track 0.26 -> 8.36 mm
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- removed copper zone on B.Cu, net GND_L
- removed copper zone on F.Cu, net GND_L
Other:
- board size 255.3 x 104.6 mm -> 124.8 x 104.5 mm
