File: pcb-left/pcb-left.kicad_pcb (KiCad board)
At the start: 2 copper layers, 124.8 x 104.5 mm, 43 parts, among them J1 BAT, U1 xiao-ble

Commit message: Update schematic and pcb to rev 0.32
Parts:
- J1: footprint karmalib:JST_PH_S2B-PH-SM4-TB -> Connector_JST:JST_PH_S2B-PH-SM4-TB_1x02-1MP_P2.00mm_Horizontal
Connections:
- J1 pad 1: VBAT_L -> GND_L
- J1 pad 2: GND_L -> VBAT_L
Routing:
- net VBAT_L: track 75.2 -> 74.4 mm
