File: pcb-right/pcb-right.kicad_pcb (KiCad board)
At the start: 2 copper layers, 124.8 x 104.5 mm, 43 parts, among them J2 BAT, U2 xiao-ble

Commit message: Update schematic and pcb to rev 0.32
Parts:
- J2: footprint karmalib:JST_PH_S2B-PH-SM4-TB -> Connector_JST:JST_PH_S2B-PH-SM4-TB_1x02-1MP_P2.00mm_Horizontal
Connections:
- J2 pad 1: VBAT_R -> GND_R
- J2 pad 2: GND_R -> VBAT_R
Routing:
- net VBAT_R: track 82.5 -> 83.3 mm
